File: Hardware/Multirotor_ESC/component_sheets/voltage_regulation.kicad_sch (KiCad schematic)
At the start: 18 parts

Commit message: Improve signage and sheet descriptions
Other:
- company: (none) -> Thomas Francois & Missouri S&T Multirotor Design Team
- title: (none) -> Multirotor ESC Board
Changed lines of the file:
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@@
 (kicad_sch (version 20211123) (generator eeschema)
   (paper "A4")
+  (title_block
+    (title "Multirotor ESC Board")
+    (date "2022-09-12")
+    (rev "v0.0.1")
+    (company "Thomas Francois & Missouri S&T Multirotor Design Team")
+    (comment 1 "Demonstration of example ESC board")
+    (comment 2 "Based upon Phil's Lab Video Demonstration")
+    (comment 3 "ESC Hardware Design (1/2) - Phil's Lab #66")
+    (comment 4 "https://www.youtube.com/watch?v=dJjxcjJOlN0")
+  )
   (junction (at 202.565 61.595) (diameter 0) (color 0 0 0 0)
   )
