File: Hardware/Multirotor_ESC/component_sheets/inverter.kicad_sch (KiCad schematic)
At the start: 18 parts

Commit message: Reorganized sheets
Parts:
- removed C?: 47μF, symbol Device:C
- removed C? (x2): 1μF, symbol Device:C
- removed C?: 1nF, symbol Device:C
- removed C?: 100nF, symbol Device:C
- removed C?: 10nF, symbol Device:C
- removed D?: D_TVS, symbol Device:D_TVS
- removed D?: D_Schottky, symbol Device:D_Schottky
- removed Q? (x2): SIR182DP-T1-RE3, symbol Transistor_FET:IRL6283M
- removed R?: 4.7kΩ, symbol Device:R_US
- removed R? (x2): 100Ω, symbol Device:R_US
- removed R?: 2mΩ, symbol Device:R_US
- removed R? (x2): 1kΩ, symbol Device:R_US
- removed U?: INA180, Package_TO_SOT_SMD:SOT-23-5, symbol Amplifier_Current:INA169
- removed U?: IR2103, symbol Driver_FET:IR2103
- added C? (x2): 1μF, symbol Device:C
- added C?: 47μF, symbol Device:C
- added C?: 10nF, symbol Device:C
- added C?: 1nF, symbol Device:C
- added C?: 100nF, symbol Device:C
- added D?: D_TVS, symbol Device:D_TVS
- added D?: D_Schottky, symbol Device:D_Schottky
- added Q? (x2): SIR182DP-T1-RE3, symbol Transistor_FET:IRL6283M
- added R? (x2): 100Ω, symbol Device:R_US
- added R?: 4.7kΩ, symbol Device:R_US
- added R? (x2): 1kΩ, symbol Device:R_US
- added R?: 2mΩ, symbol Device:R_US
- added U?: INA180, Package_TO_SOT_SMD:SOT-23-5, symbol Amplifier_Current:INA169
- added U?: IR2103, symbol Driver_FET:IR2103
Connections:
- net +3V3: now also C?.2, U?.5 (V+)
- net +BATT: now also C?.1, C?.2, D?.2 (A), Q?.1 (D), U?.1 (VCC)
- net GND: now also C?.1, C?.1, C?.1, C?.1, C?.2, D?.1 (A1), R?.1, R?.2, U?.2 (GND), U?.4 (-), U?.4 (COM)
- net HIN: now also U?.2 (HIN)
- net SENSE_I: now also C?.2, R?.1
- net SENSE_V: now also C?.2, R?.1, R?.1
- net VIS: now also R?.2, U?.1
- net VPH: now also C?.2, D?.2 (A2), Q?.1 (D), Q?.3 (S), R?.2, U?.6 (VS)
- net VPH_RS: now also Q?.3 (S), R?.2, U?.3 (+)
- net V_HO: now also R?.1, U?.7 (HO)
- net V_LO: now also R?.1, U?.5 (LO)
- net ~{LIN}: now also U?.3 (~{LIN})
- new net: Q?.2 (G), R?.2 (x2)
- new net: C?.1, D?.1 (K), U?.8 (VB)

Commit message: Improve signage and sheet descriptions
Other:
- note added: "AC Half-Bridge Inverter - Single Phase"
- note removed: "AC Inverter - Single Phase"
- company: (none) -> Thomas Francois & Missouri S&T Multirotor Design Team
- title: (none) -> Multirotor ESC Board - AC Half Bridge Inverter
Changed lines of the file:
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@@
 (kicad_sch (version 20211123) (generator eeschema)
   (paper "A4")
+  (title_block
+    (title "Multirotor ESC Board - AC Half Bridge Inverter")
+    (date "2022-09-12")
+    (rev "v0.0.1")
+    (company "Thomas Francois & Missouri S&T Multirotor Design Team")
+    (comment 1 "Demonstration of example ESC board")
+    (comment 2 "Based upon Phil's Lab Video Demonstration")
+    (comment 3 "ESC Hardware Design (1/2) - Phil's Lab #66")
+    (comment 4 "https://www.youtube.com/watch?v=dJjxcjJOlN0")
+  )
   (junction (at 113.03 78.105) (diameter 0) (color 0 0 0 0)
   )
@@
     (effects (font (size 1.27 1.27)) (justify left bottom))
   )
-  (text "AC Inverter - Single Phase" (at 33.655 48.26 0)
+  (text "AC Half-Bridge Inverter - Single Phase" (at 33.655 48.26 0)
     (effects (font (size 5.08 5.08)) (justify left bottom))
   )

Commit message: Improved component sheet labels
Connections:
- net SENSE_I renamed I_SENSE
- net SENSE_V renamed V_SENSE
Changed lines of the file:
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@@
     (effects (font (size 1.27 1.27)) (justify right))
   )
-  (hierarchical_label "SENSE_V" (shape output) (at 231.775 128.27 0)
+  (hierarchical_label "V_SENSE" (shape output) (at 231.775 128.27 0)
     (effects (font (size 1.27 1.27)) (justify left))
   )
-  (hierarchical_label "SENSE_I" (shape output) (at 191.77 128.27 0)
+  (hierarchical_label "I_SENSE" (shape output) (at 191.77 128.27 0)
     (effects (font (size 1.27 1.27)) (justify left))
   )
